File: VGA2NTSCv11-jnftech.sch (KiCad schematic (older format))
At the start: 50 parts, among them J1 RCA Yellow, J3 MD-40SM, J4 SCART Female, J5 RCA White, J6 RCA Red, J7 Micro USB, U1 Video Buffer, U2 Encoder, U3 OSC/DIV, X1 XTAL

Commit message: Cleanup associations between schematic, PCB, and Netlist
Parts:
- C6, C9: footprint VGA2NTSC:CP_Tantalum_Case-D_EIA-7343-31_Wave-JFT -> VGA2NTSC:CP_Tantalum_Case-C_EIA-6032-28_JFT
- U1: footprint Housings_SSOP:TSSOP-14_4.4x5mm_Pitch0.65mm -> VGA2NTSC:TSSOP-14_4.4x5mm_Pitch0.65mm-JFT
- U2: footprint Housings_SOIC:SOIC-16W_7.5x10.3mm_Pitch1.27mm -> VGA2NTSC:SOIC-16W_7.5x10.3mm_Pitch1.27mm_HS
- U3: footprint Housings_SOIC:SOIC-8_3.9x4.9mm_Pitch1.27mm -> VGA2NTSC:SOIC-8_3.9x4.9mm_Pitch1.27mm-JFT
Changed lines of the file:
@@
 F 0 "U3" H 8750 5250 60  0000 L BNN
 F 1 "OSC/DIV" H 8750 4650 60  0000 L BNN
-F 2 "Housings_SOIC:SOIC-8_3.9x4.9mm_Pitch1.27mm" H 8750 4650 60  0001 C CNN
+F 2 "VGA2NTSC:SOIC-8_3.9x4.9mm_Pitch1.27mm-JFT" H 8750 4650 60  0001 C CNN
 F 3 "" H 8750 4650 60  0000 C CNN
 	1    9150 5000
@@
 F 0 "U2" H 4050 5150 60  0000 L BNN
 F 1 "Encoder" H 4050 3950 60  0000 L BNN
-F 2 "Housings_SOIC:SOIC-16W_7.5x10.3mm_Pitch1.27mm" H 4050 3950 60  0001 C CNN
+F 2 "VGA2NTSC:SOIC-16W_7.5x10.3mm_Pitch1.27mm_HS" H 4050 3950 60  0001 C CNN
 F 3 "" H 4050 3950 60  0000 C CNN
 	1    3750 4950
@@
 F 0 "C6" V 13040 3960 60  0000 R TNN
 F 1 "Cap 100uF 1210" V 12760 3960 60  0000 R TNN
-F 2 "VGA2NTSC:CP_Tantalum_Case-D_EIA-7343-31_Wave-JFT" H 12760 3960 60  0001 C CNN
+F 2 "VGA2NTSC:CP_Tantalum_Case-C_EIA-6032-28_JFT" H 12760 3960 60  0001 C CNN
 F 3 "" H 12760 3960 60  0000 C CNN
 	1    13050 3950
@@
 F 0 "C9" V 13040 4460 60  0000 R TNN
 F 1 "Cap 100uF 1210" V 12760 4460 60  0000 R TNN
-F 2 "VGA2NTSC:CP_Tantalum_Case-D_EIA-7343-31_Wave-JFT" H 12760 4460 60  0001 C CNN
+F 2 "VGA2NTSC:CP_Tantalum_Case-C_EIA-6032-28_JFT" H 12760 4460 60  0001 C CNN
 F 3 "" H 12760 4460 60  0000 C CNN
 	1    13050 4450
@@
 F 0 "U1" H 8350 3550 60  0000 L BNN
 F 1 "Video Buffer" H 8350 2650 60  0000 L BNN
-F 2 "Housings_SSOP:TSSOP-14_4.4x5mm_Pitch0.65mm" H 8350 2650 60  0001 C CNN
+F 2 "VGA2NTSC:TSSOP-14_4.4x5mm_Pitch0.65mm-JFT" H 8350 2650 60  0001 C CNN
 F 3 "" H 8350 2650 60  0000 C CNN
 	1    8850 3150

Commit message: Updating project to 20210703 version
Parts:
- added C21, C22, C23, C24, C25: Cap 220uf Case C, VGA2NTSC:CP_Tantalum_Case-C_EIA-6032-28_JFT, symbol Device:CP_Small
- added JP1, JP2: Jumper_NO_Small, VGA2NTSC:WirepadJumperSm, symbol Device:Jumper_NO_Small
- added P1: EXT_CLOCK, VGA2NTSC:TH_Hole_One_1mm, symbol VGA2NTSC-v11-rescue:wirepad
- added P2: EXT_STD_TOGGLE, VGA2NTSC:Pin_Header_Straight_1x03_Pitch2.54mm_NoSilk, symbol Connector:Conn_01x03_Female
- added P3: YTRAP_FEED, VGA2NTSC:TH_Hole_One_1mm, symbol VGA2NTSC-v11-rescue:wirepad
- added P4: VCC_TAP, VGA2NTSC:TH_Hole_One_1mm, symbol VGA2NTSC-v11-rescue:wirepad
- added P5: GND_TAP, VGA2NTSC:TH_Hole_One_1mm, symbol VGA2NTSC-v11-rescue:wirepad
- added SW1: SW_SPDT, VGA2NTSC:SW_HRO-SK-12D02_SPDT_Angled, symbol Switch:SW_SPDT
- C1, C10, C11, C12, C16, C2, C3, C4, C5, C7, C8: symbol VGA2NTSC-v11-rescue:Cap_0.1uF_0402- -> Device:C
- C13, C14: value Cap 10uF 0603 -> 10uf; symbol VGA2NTSC-v11-rescue:Cap_10uF_0603- -> Device:C
- C15: symbol VGA2NTSC-v11-rescue:Cap_10uF_0603- -> Device:C
- C17: symbol VGA2NTSC-v11-rescue:Cap_18pF_0402- -> Device:C
- C18, C19, C20: symbol VGA2NTSC-v11-rescue:Cap_47pF- -> Device:C
- C6, C9: value Cap 100uF 1210 -> Cap 220uf Case C; symbol VGA2NTSC-v11-rescue:Cap_100uF_1210- -> Device:CP_Small
- J1, J5, J6: footprint VGA2NTSC:RCJ-04x -> VGA2NTSC:RCJ-04x_NoHole
- J4: footprint VGA2NTSC:SCART-F-RA-Pin11centerNPTH -> VGA2NTSC:SCART-F-RA-NoHole
- R1, R10, R2, R3, R4, R5, R6, R7, R8, R9: symbol VGA2NTSC-v11-rescue:Res_75_0402- -> Device:R
- R11, R13: value Res 1k 0402 -> 1K; symbol VGA2NTSC-v11-rescue:Res_1k_0402- -> Device:R
- R12: value Res 1M 0402 -> 1M; symbol VGA2NTSC-v11-rescue:Res_1M_0402- -> Device:R
- R14: symbol VGA2NTSC-v11-rescue:Res_4.7k_0402- -> Device:R
- R15, R16: value 49.9 -> 49R9; symbol VGA2NTSC-v11-rescue:Res_49.9_0402- -> Device:R
Connections:
- net BOUT: now also C25.2; no longer R8.2
- net CLOCK: now also JP1.1, P1.1; no longer U3.1 (OUT)
- net CSYNC_OUT: now also C22.2; no longer R2.2
- net CVBS_OUT: now also C21.2; no longer R1.2
- net GND: now also P2.1 (Pin_1), P5.1
- net GOUT: now also C24.2; no longer R7.2
- net ROUT: now also C23.2; no longer R3.2
- net VCC: now also JP2.2, P2.3 (Pin_3), P4.1; no longer U2.1 (STND)
- net VS: now also SW1.2 (B); no longer J2.14, R14.2
- net at U2.12 (YTRAP): now also P3.1
- new net: J2.14, SW1.3 (C)
- new net: R14.2, SW1.1 (A)
- new net: C21.1, R1.2
- new net: JP2.1, P2.2 (Pin_2), U2.1 (STND)
- new net: JP1.2, U3.1 (OUT)
- new net: C22.1, R2.2
- new net: C25.1, R8.2
- new net: C24.1, R7.2
- new net: C23.1, R3.2
Other:
- note added: "C21-C25 CAN BE CONSIDERED OPTIONAL AS\nPER THE ORIGINAL DESIGN THESE LINES (CVBS and RGB)\nWERE DC COUPLED, NOT AC COUPLED\nIF DC COUPLING IS DESIRED, YOU MUST JUMPER THESE PADS\n(1206 or 1812 sized 0ohm resistors will do)"
- note added: "JP1: CLOSE FOR NORMAL NTSC OPERATION\nUSING LOCAL OSC\nLEAVE OPEN TO SUPPLY EXTERNAL OSCILLATOR (P1)"
- note added: "JP2: CLOSE FOR NORMAL NTSC OPERATION\nLEAVE OPEN TO ENABLE SWITCHING BETWEEN NTSC/PAL\n(Requires external oscillator that can be fed in\n using the EXT_CLOCK pad P1)"
- note added: "P3: DEV ACCESS TO YTRAP PIN (SEE DATASHEET)\nYTRAP DOES NOT HELP SOLVE DOT CRAWL ISSUES ON CVBS"
